File: pcb/bakeneko-65-pcb.kicad_pcb (KiCad board)
At the start: 2 copper layers, 303.8 x 94.2 mm, 160 parts, among them J1 JST SH 4-pin, SW1 Reset, U1 USBLC6-2SC6, U2 ATmega32U4-AU, Y1 16MHz

Commit message: yep
Parts:
- added AdafruitLEBluetooth1: Conn_01x09_MountingPin, Connector_PinHeader_2.54mm:PinHeader_1x09_P2.54mm_Vertical, B.Cu at (92.2, 85.1)
Connections:
- U2 pad 10: Net-(U2-Pad10) -> BleCS
- U2 pad 11: Net-(U2-Pad11) -> BleIRQ
- U2 pad 41: Net-(U2-Pad41) -> (no net)
- U2 pad 42: Net-(U2-Pad42) -> (no net)
- U2 pad 9: Net-(U2-Pad9) -> BleReset

Commit message: Added hotswap
Parts:
- removed D14: 1N4148, Diode_SMD:D_SOD-123
- removed MX14, MX15, MX63: 1u, MX_Only:MXOnly-1U-NoLED
- removed MX33: 1.25u, MX_Only:MXOnly-1.25U-NoLED
- removed MX62, MX64, MX67: 1.5u, MX_Only:MXOnly-1.5U-NoLED
- removed MX65: 7u, MX_Only:MXOnly-7U-ReversedStabilizers-NoLED
- MX1, MX10, MX11, MX12, MX13, MX16, MX19, MX2, MX20, MX21, MX22, MX23, MX24, MX25, MX26, MX27, MX28, MX29, MX3, MX30, MX32, MX35, MX36, MX37, MX38, MX39, MX4, MX40, MX41, MX42, MX43, MX44, MX45, MX47, MX49, MX5, MX50, MX51, MX52, MX53, MX54, MX55, MX56, MX57, MX58, MX6, MX60, MX61, MX68, MX69, MX7, MX70, MX8, MX9: footprint MX_Only:MXOnly-1U-NoLED -> MechKeys:Kailh_socket_MX
- MX17: footprint MX_Only:MXOnly-2U-NoLED -> MX_Only:MXOnly-2U-Hotswap
- MX18, MX31: footprint MX_Only:MXOnly-1.5U-NoLED -> MX_Only:MXOnly-1.5U-Hotswap
- MX34, MX59: footprint MX_Only:MXOnly-1.75U-NoLED -> MX_Only:MXOnly-1.75U-Hotswap
- MX46, MX48: footprint MX_Only:MXOnly-2.25U-NoLED -> MX_Only:MXOnly-2.25U-Hotswap
- MX66, MX71, MX72, MX73, MX75: footprint MX_Only:MXOnly-1.25U-NoLED -> MX_Only:MXOnly-1.25U-Hotswap
- MX74: footprint MX_Only:MXOnly-6.25U-ReversedStabilizers-NoLED -> MX_Only:MXOnly-6.25U-Hotswap-ReversedStabilizers
Routing:
- net (no net): track 0.00 -> 1107.0 mm
- net COL6: track 212.1 -> 113.1 mm
- net COL9: track 265.0 -> 169.0 mm
- net COL2: track 143.7 -> 52.2 mm
- net COL13: track 353.1 -> 263.0 mm
- net COL1: track 109.3 -> 19.2 mm
- net COL11: track 293.6 -> 205.0 mm
- net COL12: track 318.3 -> 232.2 mm
- net COL15: track 355.0 -> 278.6 mm
- net COL5: track 161.8 -> 94.8 mm
- net COL4: track 143.4 -> 76.4 mm
- net COL8: track 217.4 -> 150.4 mm
- net COL7: track 198.8 -> 131.7 mm
- net COL3: track 125.1 -> 58.1 mm
- net COL10: track 254.7 -> 187.6 mm
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
Commit message: finished keyboard pcb
Parts:
- removed AdafruitLEBluetooth1: Conn_01x09_MountingPin, Connector_PinHeader_2.54mm:PinHeader_1x09_P2.54mm_Vertical
- added J2: Conn_01x04, Connector_JST:JST_SH_BM03B-SRSS-TB_1x03-1MP_P1.00mm_Vertical, B.Cu at (171.0, 55.9)
- added J3: Prog, Connector_PinHeader_2.54mm:PinHeader_1x06_P2.54mm_Vertical, F.Cu at (3.33, 54.6)
- added J4: Liion, Connector_JST:JST_SH_BM03B-SRSS-TB_1x03-1MP_P1.00mm_Vertical, B.Cu at (150.7, 55.9)
- added J5: BLE, Connector_PinHeader_2.54mm:PinHeader_1x09_P2.54mm_Vertical, F.Cu at (92.2, 77.5)
- J1: value JST SH 4-pin -> USB
- moved C4 151.5 mm to (160.5, 92.7), turned to 0 degrees
- moved C2 144.5 mm to (157.0, 74.9), turned to 180 degrees
- moved C3 139.1 mm to (167.2, 80.0), turned to 270 degrees
- moved C5 136.8 mm to (168.0, 85.7)
- moved C6 136.8 mm to (168.0, 91.3)
- moved Y1 136.8 mm to (168.0, 88.5)
- moved U2 136.5 mm to (157.0, 83.8)
- moved F1 132.8 mm to (144.3, 85.1), turned to 270 degrees
- moved SW1 130.6 mm to (176.1, 85.1), turned to 90 degrees
- moved C7 129.5 mm to (148.1, 76.2), turned to 90 degrees
- moved R3 129.1 mm to (146.8, 86.4), turned to 270 degrees
- moved R1 128.3 mm to (169.7, 80.0)
- moved R4 127.5 mm to (151.9, 92.7), turned to 0 degrees
- moved R2 123.5 mm to (141.8, 86.4), turned to 270 degrees
- moved U1 123.1 mm to (144.3, 90.2), turned to 90 degrees
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Connections:
- J1 pad 1: VBUS -> USB_PWR
Routing:
- net (no net): track 1107.0 -> 0.00 mm
- net COL1: track 19.2 -> 217.9 mm, vias 0 -> 2
- net RESET: track 28.0 -> 217.9 mm, vias 0 -> 1
- net ROW0: track 295.9 -> 478.2 mm, vias 2 -> 4
- net BleIRQ: track 0.00 -> 178.2 mm, vias 0 -> 1
- net BleReset: track 0.00 -> 173.8 mm, vias 0 -> 1
- net BleCS: track 0.00 -> 170.9 mm
- net GND: track 138.5 -> 308.9 mm, vias 4 -> 6
- net COL14: track 318.9 -> 168.8 mm, vias 1 -> 4
- net COL2: track 52.2 -> 201.7 mm
- net ROW1: track 284.9 -> 428.0 mm, vias 2 -> 7
- net COL0: track 99.8 -> 235.4 mm, vias 1 -> 2
- net COL3: track 58.1 -> 186.7 mm, vias 0 -> 2
- net USB_PWR: track 0.00 -> 118.5 mm, vias 0 -> 3
- net +5V: track 106.9 -> 220.3 mm, vias 6 -> 4
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- removed copper zone on B.Cu, net GND
Other:
- board size 303.8 x 94.2 mm -> 304.2 x 94.2 mm
- board text removed: "Bakeneko 65 v3.0"
